Commit message: new stuff

File: Rviz/test_01/src/robot_description/urdf/robot.urdf (robot description, URDF)
Before this commit: robot origins, 3 links, 2 joints
Links:
- added link torso; visual mesh filename=package://robot_description/STL/body_link.stl scale=0.001 0.001 0.001
- link base_link: geometry 
Joints:
- added joint base_to_torso: type revolute, parent base_link, child torso, origin xyz=0 0 0.7, limit lower=-1.5708 upper=1.5708 effort=10 velocity=3

Commit message: enkoder

File: Rviz/test_01/src/robot_description/urdf/robot.urdf (robot description, URDF)
Before this commit: robot origins, 4 links, 3 joints
Joints:
- joint base_to_torso: origin xyz=0 0 0.7 -> xyz=0 0 0
